Commit message: Add files via upload

File: src/dp/urdf/dp_params.xacro (robot description, xacro)
@@ -34,4 +34,23 @@
   <xacro:property name="izz2" value="${(1.0/12.0) * mass2 * (length2 * length2 + width2 * width2) + Jm2_ef}"/> <!-- super simplificación a fines didácticos -->
   <xacro:property name="iyy2" value="${izz2}"/>
+  <!-- Parámetros del eslabón 3 -->
+  <xacro:property name="mass3" value="1.5"/>
+  <xacro:property name="length3" value="0.22"/>
+  <xacro:property name="width3" value="0.02"/>
+  <xacro:property name="a3" value="${length3 - width3}"/>
+  <xacro:property name="Jm3" value="0.0001"/>
+  <xacro:property name="N3"  value="10"/>
+  <xacro:property name="Jm3_ef" value="${N3*N3 * Jm3}"/>
+  <xacro:property name="ixx3" value="${(1.0/6.0) * mass3 * (width3 * width3)}"/>
+  <xacro:property name="izz3" value="${(1.0/12.0) * mass3 * (length3 * length3 + width3 * width3) + Jm3_ef}"/>
+  <xacro:property name="iyy3" value="${izz3}"/>
+  <!-- Argumentos para joint3 -->
+  <xacro:arg name="damping3" default="0.1"/>
+  <xacro:arg name="friction3" default="0.01"/>
+  <xacro:arg name="q3_max" default="3.14"/>
+  <xacro:arg name="q3_min" default="-3.14"/>
+  <xacro:arg name="qp3_max" default="5.0"/>
+  <xacro:arg name="tau3_max" default="100.0"/>
+  <xacro:arg name="q3_ini" default="1.0"/>
   <!-- Valores que pueden modificarse en otros archivos xacro y que funcionan como argumentos -->
   <xacro:arg name="damping1" default="0.1"/>                 <!-- rozamiento viscoso -->
